File: duin/duin.sch (KiCad schematic (older format))
At the start: 17 parts, among them IC1 ATMEGA8-PU, P1 ADC, P2 CONN_8, X1 CRYSTAL

Commit message: duin changes
Parts:
- added C7: C, symbol C
- added D2: LED, symbol LED
- added R2: R, symbol R
- gave numbers to parts that had none: 9
Connections:
- net +5V: now also P3.3, U1.VO
- net GND: now also P3.4, P3.5, C7.2, D2.2 (K)
- net at IC1.1 (PC6(/RESET)), R1.2, SW1.1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: now also P3.1
- net at IC1.19 (PB5(SCK)), P2.6 (P6): now also R2.1
- new net: D2.1 (A), R2.2
Other:
- moved on the sheet: P3
Changed lines of the file:
@@
-EESchema Schematic File Version 2  date Fri 03 Dec 2010 12:15:25 AM BRST
+EESchema Schematic File Version 2  date Fri 03 Dec 2010 12:47:36 AM BRST
 LIBS:power
 LIBS:device
@@
 $EndDescr
 Wire Wire Line
+	4500 1300 4500 1400
+Wire Wire Line
+	3500 1200 3500 1200
+Wire Wire Line
+	6000 6350 6000 6200
+Connection ~ 6650 5500
+Wire Wire Line
+	6650 5850 6650 5500
+Wire Wire Line
 	6800 3950 6000 3950
 Wire Wire Line
@@
 Connection ~ 3550 2550
 Connection ~ 3550 3050
-Wire Wire Line
-	3550 2150 3550 3050
 Connection ~ 3250 1600
 Wire Wire Line
-	3500 1600 1400 1600
-Wire Wire Line
-	3500 1200 3100 1200
+	3100 1200 4500 1200
 Connection ~ 1900 1600
 Wire Wire Line
-	1400 1600 1400 1300
+	1400 1300 1400 1600
 Wire Wire Line
 	1800 1200 2300 1200
@@
 Wire Wire Line
 	6800 4050 6000 4050
+Wire Wire Line
+	6650 6900 6650 6750
+Wire Wire Line
+	6400 5800 5700 5800
+Wire Wire Line
+	4500 1000 4050 1000
+Wire Wire Line
+	4050 1000 4050 2000
+Wire Wire Line
+	4050 2000 3550 2000
+Wire Wire Line
+	3550 2000 3550 3050
+Connection ~ 3550 2150
+Wire Wire Line
+	1400 1600 4250 1600
+Wire Wire Line
+	4250 1600 4250 1400
+Wire Wire Line
+	4250 1400 4500 1400
+Text GLabel 3500 1200 1    60   Input ~ 0
++5V
+Text GLabel 6000 6350 2    60   Input ~ 0
+GND
+$Comp
+L C C7
+U 1 1 4CF85318
+P 6000 6000
+F 0 "C7" H 6050 6100 50  0000 L CNN
+F 1 "C" H 6050 5900 50  0000 L CNN
+	1    6000 6000
+	1    0    0    -1
+$EndComp
+Text GLabel 6650 6900 2    60   Input ~ 0
+GND
+$Comp
+L LED D2
+U 1 1 4CF852E1
+P 6650 6550
+F 0 "D2" H 6650 6650 50  0000 C CNN
+F 1 "LED" H 6650 6450 50  0000 C CNN
+	1    6650 6550
+	0    1    1    0
+$EndComp
+$Comp
+L R R2
+U 1 1 4CF852D9
+P 6650 6100
+F 0 "R2" V 6730 6100 50  0000 C CNN
+F 1 "R" V 6650 6100 50  0000 C CNN
+	1    6650 6100
+	1    0    0    -1
+$EndComp
 Text GLabel 6400 5600 0    60   Input ~ 0
 GND
 $Comp
-L CONN_6 P?
+L CONN_6 P3
 U 1 1 4CF8513C
-P 4850 1300
-F 0 "P?" V 4800 1300 60  0000 C CNN
-F 1 "CONN_6" V 4900 1300 60  0000 C CNN
-	1    4850 1300
-	1    0    0    -1
-$EndComp
-$Comp
-L CONN_6 P?
+P 4850 1250
+F 0 "P3" V 4800 1250 60  0000 C CNN
+F 1 "CONN_6" V 4900 1250 60  0000 C CNN
+	1    4850 1250
+	1    0    0    -1
+$EndComp
+$Comp
+L CONN_6 P4
 U 1 1 4CF85130
 P 6750 3300
-F 0 "P?" V 6700 3300 60  0000 C CNN
+F 0 "P4" V 6700 3300 60  0000 C CNN
 F 1 "CONN_6" V 6800 3300 60  0000 C CNN
 	1    6750 3300
@@
 GND
 $Comp
-L DPST SW?
+L DPST SW1
 U 1 1 4CF85056
 P 4050 2350
-F 0 "SW?" H 4050 2450 70  0000 C CNN
+F 0 "SW1" H 4050 2450 70  0000 C CNN
 F 1 "DPST" H 4050 2250 70  0000 C CNN
 	1    4050 2350
 	1    0    0    -1
 $EndComp
-Text GLabel 3500 1600 2    60   Input ~ 0
-GND
-$Comp
-L C C?
+Text GLabel 3500 1600 1    60   Input ~ 0
+GND
+$Comp
+L C C6
 U 1 1 4CF84F42
 P 3250 1400
-F 0 "C?" H 3300 1500 50  0000 L CNN
+F 0 "C6" H 3300 1500 50  0000 L CNN
 F 1 "C" H 3300 1300 50  0000 L CNN
 	1    3250 1400
@@
 $EndComp
 $Comp
-L C C?
+L C C5
 U 1 1 4CF84F0C
 P 2200 1400
-F 0 "C?" H 2250 1500 50  0000 L CNN
+F 0 "C5" H 2250 1500 50  0000 L CNN
 F 1 "C" H 2250 1300 50  0000 L CNN
 	1    2200 1400
@@
 $EndComp
 $Comp
-L C C?
+L C C4
 U 1 1 4CF84F06
 P 1900 1400
-F 0 "C?" H 1950 1500 50  0000 L CNN
+F 0 "C4" H 1950 1500 50  0000 L CNN
 F 1 "C" H 1950 1300 50  0000 L CNN
 	1    1900 1400
@@
 $EndComp
 $Comp
-L DIODE D?
+L DIODE D1
 U 1 1 4CF84ED5
 P 1600 1200
-F 0 "D?" H 1600 1300 40  0000 C CNN
+F 0 "D1" H 1600 1300 40  0000 C CNN
 F 1 "DIODE" H 1600 1100 40  0000 C CNN
 	1    1600 1200
@@
 $EndComp
 $Comp
-L CONN_3 K?
+L CONN_3 K1
 U 1 1 4CF84EA6
 P 1050 1200
-F 0 "K?" H 1000 1250 50  0000 C CNN
+F 0 "K1" H 1000 1250 50  0000 C CNN
 F 1 "CONN_3" V 1100 1200 40  0000 C CNN
 	1    1050 1200
@@
 $EndComp
 $Comp
-L LM7805 U?
+L LM7805 U1
 U 1 1 4CF84CFD
 P 2700 1250
-F 0 "U?" H 2850 1054 60  0000 C CNN
+F 0 "U1" H 2850 1054 60  0000 C CNN
 F 1 "LM7805" H 2700 1450 60  0000 C CNN
 	1    2700 1250
@@
 Text GLabel 3300 5150 0    60   Input ~ 0
 GND
-Text GLabel 6400 5800 0    60   Input ~ 0
+Text GLabel 5700 5800 0    60   Input ~ 0
 AREF
 $Comp

Commit message: duin
Connections:
- net +5V: now also C6.1
- net at D1.2 (K), U1.VI: now also C4.1, C5.1
Changed lines of the file:
@@
-EESchema Schematic File Version 2  date Fri 03 Dec 2010 12:47:36 AM BRST
+EESchema Schematic File Version 2  date Sat 04 Dec 2010 12:32:55 AM BRST
 LIBS:power
 LIBS:device
@@
 $EndDescr
 Wire Wire Line
-	4500 1300 4500 1400
+	1800 1200 2300 1200
+Connection ~ 3250 1200
+Connection ~ 2200 1200
+Wire Wire Line
+	4250 1400 4500 1400
+Wire Wire Line
+	4250 1400 4250 1600
+Wire Wire Line
+	4250 1600 1400 1600
+Connection ~ 3550 2150
+Wire Wire Line
+	3550 3050 3550 2000
+Wire Wire Line
+	3550 2000 4050 2000
+Wire Wire Line
+	4050 2000 4050 1000
+Wire Wire Line
+	4050 1000 4500 1000
+Wire Wire Line
+	5700 5800 6400 5800
+Wire Wire Line
+	6650 6900 6650 6750
+Wire Wire Line
+	6800 4050 6000 4050
+Wire Wire Line
+	6800 4250 6000 4250
+Wire Wire Line
+	6800 4450 6000 4450
+Wire Wire Line
+	6800 4650 6000 4650
+Wire Wire Line
+	6000 4950 6650 4950
+Wire Wire Line
+	6650 4950 6650 5100
+Wire Wire Line
+	6650 5100 6800 5100
+Wire Wire Line
+	6000 5150 6550 5150
+Wire Wire Line
+	6550 5150 6550 5300
+Wire Wire Line
+	6550 5300 6800 5300
+Wire Wire Line
+	6800 5500 6450 5500
+Wire Wire Line
+	6450 5500 6450 5350
+Wire Wire Line
+	6450 5350 6000 5350
+Wire Wire Line
+	6400 5600 6800 5600
+Wire Wire Line
+	4550 2550 4550 2150
+Connection ~ 2700 1600
+Connection ~ 2200 1600
+Wire Wire Line
+	2700 1600 2700 1500
+Wire Wire Line
+	1300 1300 1400 1300
+Wire Wire Line
+	1300 1300 1300 1100
+Wire Wire Line
+	1300 1100 1400 1100
+Connection ~ 2550 3750
+Wire Wire Line
+	2400 3750 2550 3750
+Connection ~ 3600 4300
+Wire Wire Line
+	3300 4450 3300 4300
+Wire Wire Line
+	3300 4300 3600 4300
+Wire Wire Line
+	3600 5250 3600 5050
+Wire Wire Line
+	2550 3450 2550 4050
+Wire Wire Line
+	2950 3450 3250 3450
+Wire Wire Line
+	3250 3450 3250 3650
+Wire Wire Line
+	3250 3650 3600 3650
+Wire Wire Line
+	6400 3450 6000 3450
+Wire Wire Line
+	6400 3250 6000 3250
+Wire Wire Line
+	6400 3050 6000 3050
+Wire Wire Line
+	6000 3150 6400 3150
+Wire Wire Line
+	6000 3350 6400 3350
+Wire Wire Line
+	6000 3550 6400 3550
+Wire Wire Line
+	2950 4050 3250 4050
+Wire Wire Line
+	3250 4050 3250 3850
+Wire Wire Line
+	3250 3850 3600 3850
+Wire Wire Line
+	3600 4150 3600 4450
+Wire Wire Line
+	3600 5150 3300 5150
+Wire Wire Line
+	3300 5150 3300 4850
+Connection ~ 3600 5150
+Wire Wire Line
+	2850 4550 3600 4550
+Wire Wire Line
+	3600 3050 3200 3050
+Wire Wire Line
+	3200 2400 3200 2550
+Wire Wire Line
+	1400 1300 1400 1600
+Connection ~ 1900 1600
+Wire Wire Line
+	3100 1200 4500 1200
+Connection ~ 3250 1600
+Connection ~ 3550 3050
+Connection ~ 3550 2550
+Wire Wire Line
+	4700 2350 4550 2350
+Connection ~ 4550 2350
+Wire Wire Line
+	6400 5800 6400 5700
+Wire Wire Line
+	6400 5700 6800 5700
+Wire Wire Line
+	6800 5400 6500 5400
+Wire Wire Line
+	6500 5400 6500 5250
+Wire Wire Line
+	6500 5250 6000 5250
+Wire Wire Line
+	6800 5200 6600 5200
+Wire Wire Line
+	6600 5200 6600 5050
+Wire Wire Line
+	6600 5050 6000 5050
+Wire Wire Line
+	6800 5000 6700 5000
+Wire Wire Line
+	6700 5000 6700 4850
+Wire Wire Line
+	6700 4850 6000 4850
+Wire Wire Line
+	6000 4550 6800 4550
+Wire Wire Line
+	6800 4350 6000 4350
+Wire Wire Line
+	6800 4150 6000 4150
+Wire Wire Line
+	6800 3950 6000 3950
+Wire Wire Line
+	6650 5850 6650 5500
+Connection ~ 6650 5500
+Wire Wire Line
+	6000 6350 6000 6200
 Wire Wire Line
 	3500 1200 3500 1200
 Wire Wire Line
-	6000 6350 6000 6200
-Connection ~ 6650 5500
-Wire Wire Line
-	6650 5850 6650 5500
-Wire Wire Line
-	6800 3950 6000 3950
-Wire Wire Line
-	6800 4150 6000 4150
-Wire Wire Line
-	6800 4350 6000 4350
-Wire Wire Line
-	6000 4550 6800 4550
-Wire Wire Line
-	6000 4850 6700 4850
-Wire Wire Line
-	6700 4850 6700 5000
-Wire Wire Line
-	6700 5000 6800 5000
-Wire Wire Line
-	6000 5050 6600 5050
-Wire Wire Line
-	6600 5050 6600 5200
-Wire Wire Line
-	6600 5200 6800 5200
-Wire Wire Line
-	6000 5250 6500 5250
-Wire Wire Line
-	6500 5250 6500 5400
-Wire Wire Line
-	6500 5400 6800 5400
-Wire Wire Line
-	6800 5700 6400 5700
-Wire Wire Line
-	6400 5700 6400 5800
-Connection ~ 4550 2350
-Wire Wire Line
-	4700 2350 4550 2350
-Connection ~ 3550 2550
-Connection ~ 3550 3050
-Connection ~ 3250 1600
-Wire Wire Line
-	3100 1200 4500 1200
-Connection ~ 1900 1600
-Wire Wire Line
-	1400 1300 1400 1600
-Wire Wire Line
-	1800 1200 2300 1200
-Wire Wire Line
-	3200 2400 3200 2550
-Wire Wire Line
-	3600 3050 3200 3050
-Wire Wire Line
-	2850 4550 3600 4550
-Connection ~ 3600 5150
-Wire Wire Line
-	3300 4850 3300 5150
-Wire Wire Line
-	3300 5150 3600 5150
-Wire Wire Line
-	3600 4150 3600 4450
-Wire Wire Line
-	3600 3850 3250 3850
-Wire Wire Line
-	3250 3850 3250 4050
-Wire Wire Line
-	3250 4050 2950 4050
-Wire Wire Line
-	6000 3550 6400 3550
-Wire Wire Line
-	6000 3350 6400 3350
-Wire Wire Line
-	6000 3150 6400 3150
-Wire Wire Line
-	6400 3050 6000 3050
-Wire Wire Line
-	6400 3250 6000 3250
-Wire Wire Line
-	6400 3450 6000 3450
-Wire Wire Line
-	3600 3650 3250 3650
-Wire Wire Line
-	3250 3650 3250 3450
-Wire Wire Line
-	3250 3450 2950 3450
-Wire Wire Line
-	2550 3450 2550 4050
-Wire Wire Line
-	3600 5250 3600 5050
-Wire Wire Line
-	3600 4300 3300 4300
-Wire Wire Line
-	3300 4300 3300 4450
-Connection ~ 3600 4300
-Wire Wire Line
-	2400 3750 2550 3750
-Connection ~ 2550 3750
-Wire Wire Line
-	1400 1100 1300 1100
-Wire Wire Line
-	1300 1100 1300 1300
-Wire Wire Line
-	1300 1300 1400 1300
-Wire Wire Line
-	2700 1600 2700 1500
-Connection ~ 2200 1600
-Connection ~ 2700 1600
-Wire Wire Line
-	4550 2550 4550 2150
-Wire Wire Line
-	6400 5600 6800 5600
-Wire Wire Line
-	6000 5350 6450 5350
-Wire Wire Line
-	6450 5350 6450 5500
-Wire Wire Line
-	6450 5500 6800 5500
-Wire Wire Line
-	6800 5300 6550 5300
-Wire Wire Line
-	6550 5300 6550 5150
-Wire Wire Line
-	6550 5150 6000 5150
-Wire Wire Line
-	6800 5100 6650 5100
-Wire Wire Line
-	6650 5100 6650 4950
-Wire Wire Line
-	6650 4950 6000 4950
-Wire Wire Line
-	6800 4650 6000 4650
-Wire Wire Line
-	6800 4450 6000 4450
-Wire Wire Line
-	6800 4250 6000 4250
-Wire Wire Line
-	6800 4050 6000 4050
-Wire Wire Line
-	6650 6900 6650 6750
-Wire Wire Line
-	6400 5800 5700 5800
-Wire Wire Line
-	4500 1000 4050 1000
-Wire Wire Line
-	4050 1000 4050 2000
-Wire Wire Line
-	4050 2000 3550 2000
-Wire Wire Line
-	3550 2000 3550 3050
-Connection ~ 3550 2150
-Wire Wire Line
-	1400 1600 4250 1600
-Wire Wire Line
-	4250 1600 4250 1400
-Wire Wire Line
-	4250 1400 4500 1400
+	4500 1400 4500 1300
+Wire Wire Line
+	1900 1200 1850 1200
+Connection ~ 1900 1200
 Text GLabel 3500 1200 1    60   Input ~ 0
 +5V

Commit message: sweet, new 3d modules...
Parts:
- removed D1: DIODE, symbol DIODE
- added C8, C9: C, symbol C
- added D3: BRIDGE, symbol BRIDGE
- added U2: LD2903, symbol LM7805
Connections:
- net GND: now also C8.2, C9.2, D3.1 (-), U2.GND; no longer C4.2, K1.1 (P1), K1.3 (P3)
- net RESET: now reaches IC1.1 (PC6(/RESET)), P3.1, R1.2, SW1.1, SW1.3
- net at C5.1, U1.VI: now also D3.3 (+); no longer C4.1
- net at K1.2 (PM): now also C4.1, K1.3 (P3), D3.4
- new net: C4.2, D3.2, K1.1 (P1)
- new net: C8.1, U2.VI
- new net: C9.1, U2.VO
Other:
- moved on the sheet: C4, C5, C6, K1, P3, U1
Changed lines of the file:
@@
-EESchema Schematic File Version 2  date Sat 04 Dec 2010 12:32:55 AM BRST
+EESchema Schematic File Version 2  date Sat 04 Dec 2010 11:45:20 AM BRST
 LIBS:power
 LIBS:device
@@
 Sheet 1 1
 Title ""
-Date "3 dec 2010"
+Date "4 dec 2010"
 Rev ""
 Comp ""
@@
 $EndDescr
 Wire Wire Line
-	1800 1200 2300 1200
-Connection ~ 3250 1200
-Connection ~ 2200 1200
-Wire Wire Line
-	4250 1400 4500 1400
-Wire Wire Line
-	4250 1400 4250 1600
-Wire Wire Line
-	4250 1600 1400 1600
+	4600 1150 3350 1150
+Connection ~ 1300 950
+Wire Wire Line
+	1300 950  650  950
+Wire Wire Line
+	8900 3000 8900 3200
+Wire Wire Line
+	8500 3100 9300 3100
+Connection ~ 1300 1050
+Wire Wire Line
+	2500 550  1300 550
+Wire Wire Line
+	1300 550  1300 1150
+Wire Wire Line
+	3350 1150 3350 1400
+Connection ~ 5550 1150
+Connection ~ 4500 1150
+Wire Wire Line
+	6550 1350 6800 1350
+Wire Wire Line
+	6550 1350 6550 1550
 Connection ~ 3550 2150
 Wire Wire Line
@@
 	3550 2000 4050 2000
 Wire Wire Line
-	4050 2000 4050 1000
-Wire Wire Line
-	4050 1000 4500 1000
+	6350 950  6800 950
 Wire Wire Line
 	5700 5800 6400 5800
@@
 	6400 5600 6800 5600
 Wire Wire Line
-	4550 2550 4550 2150
-Connection ~ 2700 1600
-Connection ~ 2200 1600
-Wire Wire Line
-	2700 1600 2700 1500
-Wire Wire Line
-	1300 1300 1400 1300
-Wire Wire Line
-	1300 1300 1300 1100
-Wire Wire Line
-	1300 1100 1400 1100
+	4550 2150 4550 2550
+Connection ~ 5000 1550
+Connection ~ 4500 1550
+Wire Wire Line
+	5000 1550 5000 1450
 Connection ~ 2550 3750
 Wire Wire Line
@@
 	3300 4300 3600 4300
 Wire Wire Line
-	3600 5250 3600 5050
-Wire Wire Line
-	2550 3450 2550 4050
+	3600 5050 3600 5250
+Wire Wire Line
+	2550 4050 2550 3450
 Wire Wire Line
 	2950 3450 3250 3450
@@
 	3250 3850 3600 3850
 Wire Wire Line
-	3600 4150 3600 4450
+	3600 4450 3600 4150
 Wire Wire Line
 	3600 5150 3300 5150
@@
 	2850 4550 3600 4550
 Wire Wire Line
-	3600 3050 3200 3050
+	3200 3050 3600 3050
 Wire Wire Line
 	3200 2400 3200 2550
-Wire Wire Line
-	1400 1300 1400 1600
-Connection ~ 1900 1600
-Wire Wire Line
-	3100 1200 4500 1200
-Connection ~ 3250 1600
+Connection ~ 4200 1550
+Wire Wire Line
+	6800 1150 5400 1150
+Connection ~ 5550 1550
 Connection ~ 3550 3050
 Connection ~ 3550 2550
@@
 	6000 6350 6000 6200
 Wire Wire Line
-	3500 1200 3500 1200
-Wire Wire Line
-	4500 1400 4500 1300
-Wire Wire Line
-	1900 1200 1850 1200
-Connection ~ 1900 1200
-Text GLabel 3500 1200 1    60   Input ~ 0
+	5800 1150 5800 1150
+Wire Wire Line
+	6800 1350 6800 1250
+Connection ~ 4200 1150
+Wire Wire Line
+	1650 1400 1650 1550
+Connection ~ 1650 1550
+Wire Wire Line
+	1650 1550 6550 1550
+Wire Wire Line
+	1300 1250 1300 2250
+Wire Wire Line
+	1300 2250 2500 2250
+Connection ~ 8900 3100
+Wire Wire Line
+	650  1350 1300 1350
+Connection ~ 1300 1350
+Text GLabel 8900 3200 3    60   Input ~ 0
+GND
+Text GLabel 4050 2000 2    60   Input ~ 0
+RESET
+Text GLabel 6350 950  0    60   Input ~ 0
+RESET
+$Comp
+L C C9
+U 1 1 4CFA4448
+P 9300 2900
+F 0 "C9" H 9350 3000 50  0000 L CNN
+F 1 "C" H 9350 2800 50  0000 L CNN
+	1    9300 2900
+	1    0    0    -1
+$EndComp
+$Comp
+L C C8
+U 1 1 4CFA4444
+P 8500 2900
+F 0 "C8" H 8550 3000 50  0000 L CNN
+F 1 "C" H 8550 2800 50  0000 L CNN
+	1    8500 2900
+	1    0    0    -1
+$EndComp
+$Comp
+L LM7805 U2
+U 1 1 4CFA4437
+P 8900 2750
+F 0 "U2" H 9050 2554 60  0000 C CNN
+F 1 "LD2903" H 8900 2950 60  0000 C CNN
+	1    8900 2750
+	1    0    0    -1
+$EndComp
+$Comp
+L BRIDGE D3
+U 1 1 4CFA4424
+P 2500 1400
+F 0 "D3" H 2500 1450 70  0000 C CNN
+F 1 "BRIDGE" H 2500 1350 70  0000 C CNN
+	1    2500 1400
+	1    0    0    -1
+$EndComp
+Text GLabel 5800 1150 1    60   Input ~ 0
 +5V
 Text GLabel 6000 6350 2    60   Input ~ 0
@@
 L CONN_6 P3
 U 1 1 4CF8513C
-P 4850 1250
-F 0 "P3" V 4800 1250 60  0000 C CNN
-F 1 "CONN_6" V 4900 1250 60  0000 C CNN
-	1    4850 1250
+P 7150 1200
+F 0 "P3" V 7100 1200 60  0000 C CNN
+F 1 "CONN_6" V 7200 1200 60  0000 C CNN
+	1    7150 1200
 	1    0    0    -1
 $EndComp
@@
 	1    0    0    -1
 $EndComp
-Text GLabel 3500 1600 1    60   Input ~ 0
+Text GLabel 5800 1550 1    60   Input ~ 0
 GND
 $Comp
 L C C6
 U 1 1 4CF84F42
-P 3250 1400
-F 0 "C6" H 3300 1500 50  0000 L CNN
-F 1 "C" H 3300 1300 50  0000 L CNN
-	1    3250 1400
+P 5550 1350
+F 0 "C6" H 5600 1450 50  0000 L CNN
+F 1 "C" H 5600 1250 50  0000 L CNN
+	1    5550 1350
 	1    0    0    -1
 $EndComp
@@
 L C C5
 U 1 1 4CF84F0C
-P 2200 1400
-F 0 "C5" H 2250 1500 50  0000 L CNN
-F 1 "C" H 2250 1300 50  0000 L CNN
-	1    2200 1400
+P 4500 1350
+F 0 "C5" H 4550 1450 50  0000 L CNN
+F 1 "C" H 4550 1250 50  0000 L CNN
+	1    4500 1350
 	1    0    0    -1
 $EndComp
@@
 L C C4
 U 1 1 4CF84F06
-P 1900 1400
-F 0 "C4" H 1950 1500 50  0000 L CNN
-F 1 "C" H 1950 1300 50  0000 L CNN
-	1    1900 1400
-	1    0    0    -1
-$EndComp
-$Comp
-L DIODE D1
-U 1 1 4CF84ED5
-P 1600 1200
-F 0 "D1" H 1600 1300 40  0000 C CNN
-F 1 "DIODE" H 1600 1100 40  0000 C CNN
-	1    1600 1200
+P 650 1150
+F 0 "C4" H 700 1250 50  0000 L CNN
+F 1 "C" H 700 1050 50  0000 L CNN
+	1    650  1150
 	1    0    0    -1
 $EndComp
@@
 L CONN_3 K1
 U 1 1 4CF84EA6
-P 1050 1200
-F 0 "K1" H 1000 1250 50  0000 C CNN
-F 1 "CONN_3" V 1100 1200 40  0000 C CNN
-	1    1050 1200
+P 950 1150
+F 0 "K1" H 900 1200 50  0000 C CNN
+F 1 "CONN_3" V 1000 1150 40  0000 C CNN
+	1    950  1150
 	-1   0    0    1
 $EndComp
@@
 L LM7805 U1
 U 1 1 4CF84CFD
-P 2700 1250
-F 0 "U1" H 2850 1054 60  0000 C CNN
-F 1 "LM7805" H 2700 1450 60  0000 C CNN
-	1    2700 1250
-	1    0    0    -1
-$EndComp
+P 5000 1200
+F 0 "U1" H 5150 1004 60  0000 C CNN
+F 1 "LM7805" H 5000 1400 60  0000 C CNN
+	1    5000 1200
+	1    0    0    -1
+$EndComp

Commit message: almost finished
Parts:
- added P5: CONN_3X2, symbol CONN_3X2
- C5, C6: symbol C -> CP1
Connections:
- net +5V: now also C8.1, U2.VI; no longer IC1.20 (AVCC)
- net AREF: now also C7.1
- net GND: no longer C7.2
- net +3.3V: now reaches P3.2
- net +3.3V: now also C7.2, C9.1, IC1.20 (AVCC), U2.VO
Other:
- moved on the sheet: C8, C9, U2
Changed lines of the file:
@@
-EESchema Schematic File Version 2  date Sat 04 Dec 2010 11:45:20 AM BRST
+EESchema Schematic File Version 2  date Sun 05 Dec 2010 12:27:05 AM BRST
 LIBS:power
 LIBS:device
@@
 Sheet 1 1
 Title ""
-Date "4 dec 2010"
+Date "5 dec 2010"
 Rev ""
 Comp ""
@@
 Comment4 ""
 $EndDescr
+Text GLabel 6650 1050 0    60   Input ~ 0
++3.3V
+Wire Wire Line
+	6650 1050 6800 1050
+Connection ~ 6000 6200
+Connection ~ 6000 5800
+Wire Wire Line
+	9500 1000 9350 1000
 Wire Wire Line
 	4600 1150 3350 1150
@@
 	1300 950  650  950
 Wire Wire Line
-	8900 3000 8900 3200
-Wire Wire Line
-	8500 3100 9300 3100
+	8950 1500 8950 1300
+Wire Wire Line
+	9350 1400 8550 1400
 Connection ~ 1300 1050
 Wire Wire Line
@@
 	6400 5600 6800 5600
 Wire Wire Line
-	4550 2150 4550 2550
+	4550 2550 4550 2150
 Connection ~ 5000 1550
 Connection ~ 4500 1550
@@
 Wire Wire Line
 	2400 3750 2550 3750
-Connection ~ 3600 4300
-Wire Wire Line
-	3300 4450 3300 4300
-Wire Wire Line
-	3300 4300 3600 4300
-Wire Wire Line
-	3600 5050 3600 5250
-Wire Wire Line
-	2550 4050 2550 3450
+Connection ~ 3600 4150
+Wire Wire Line
+	3300 4450 3300 4150
+Wire Wire Line
+	3300 4150 3600 4150
+Wire Wire Line
+	3600 5250 3600 5050
+Wire Wire Line
+	2550 3450 2550 4050
 Wire Wire Line
 	2950 3450 3250 3450
@@
 Wire Wire Line
 	3250 3850 3600 3850
-Wire Wire Line
-	3600 4450 3600 4150
 Wire Wire Line
 	3600 5150 3300 5150
@@
 	2850 4550 3600 4550
 Wire Wire Line
-	3200 3050 3600 3050
+	3600 3050 3200 3050
 Wire Wire Line
 	3200 2400 3200 2550
 Connection ~ 4200 1550
 Wire Wire Line
-	6800 1150 5400 1150
+	5400 1150 6800 1150
 Connection ~ 5550 1550
 Connection ~ 3550 3050
@@
 Wire Wire Line
 	1300 2250 2500 2250
-Connection ~ 8900 3100
+Connection ~ 8950 1400
 Wire Wire Line
 	650  1350 1300 1350
 Connection ~ 1300 1350
-Text GLabel 8900 3200 3    60   Input ~ 0
+Wire Wire Line
+	8350 1000 8550 1000
+Wire Wire Line
+	3500 4350 3500 4450
+Wire Wire Line
+	3500 4450 3600 4450
+Text GLabel 3500 4350 1    60   Input ~ 0
++3.3V
+$Comp
+L CONN_3X2 P5
+U 1 1 4CFAF0AE
+P 8550 2800
+F 0 "P5" H 8550 3050 50  0000 C CNN
+F 1 "CONN_3X2" V 8550 2850 40  0000 C CNN
+	1    8550 2800
+	1    0    0    -1
+$EndComp
+Text GLabel 9500 1000 2    60   Input ~ 0
++3.3V
+Text GLabel 8350 1000 0    60   Input ~ 0
++5V
+Text GLabel 8950 1500 3    60   Input ~ 0
 GND
 Text GLabel 4050 2000 2    60   Input ~ 0
@@
 L C C9
 U 1 1 4CFA4448
-P 9300 2900
-F 0 "C9" H 9350 3000 50  0000 L CNN
-F 1 "C" H 9350 2800 50  0000 L CNN
-	1    9300 2900
+P 9350 1200
+F 0 "C9" H 9400 1300 50  0000 L CNN
+F 1 "C" H 9400 1100 50  0000 L CNN
+	1    9350 1200
 	1    0    0    -1
 $EndComp
@@
 L C C8
 U 1 1 4CFA4444
-P 8500 2900
-F 0 "C8" H 8550 3000 50  0000 L CNN
-F 1 "C" H 8550 2800 50  0000 L CNN
-	1    8500 2900
+P 8550 1200
+F 0 "C8" H 8600 1300 50  0000 L CNN
+F 1 "C" H 8600 1100 50  0000 L CNN
+	1    8550 1200
 	1    0    0    -1
 $EndComp
@@
 L LM7805 U2
 U 1 1 4CFA4437
-P 8900 2750
-F 0 "U2" H 9050 2554 60  0000 C CNN
-F 1 "LD2903" H 8900 2950 60  0000 C CNN
-	1    8900 2750
+P 8950 1050
+F 0 "U2" H 9100 854 60  0000 C CNN
+F 1 "LD2903" H 8950 1250 60  0000 C CNN
+	1    8950 1050
 	1    0    0    -1
 $EndComp
@@
 +5V
 Text GLabel 6000 6350 2    60   Input ~ 0
-GND
++3.3V
 $Comp
 L C C7
@@
 GND
 $Comp
-L C C6
+L CP1 C6
 U 1 1 4CF84F42
 P 5550 1350
@@
 $EndComp
 $Comp
-L C C5
+L CP1 C5
 U 1 1 4CF84F0C
 P 4500 1350

Commit message: duin with usb
Parts:
- removed K1: CONN_3, symbol CONN_3
- added C10: CP, symbol CP
- added D4, D5: ZENER, symbol ZENER
- added K1: JACK_2P, symbol JACK_2P
- added P6: USB, symbol CONN_4
- added P7: CONN_2, symbol CONN_2
- added R3: 1K5, symbol R
- added R4: 1M, symbol R
- added R5, R6: 68R, symbol R
Connections:
- net +3.3V: now also C7.1; no longer C7.2
- net AREF: now also C7.2; no longer C7.1
- net GND: now also C10.2, D4.1 (A), D5.1 (A), P6.4 (P4), P7.2 (PM), R4.1
- net PD2: now reaches IC1.4 (PD2(INT0)), P1.3 (P3)
- net PD2: now also R6.1
- net PD4: now reaches IC1.6 (PD4(T0/XCK)), P1.5 (P5)
- net PD4: now also R5.1
- net at IC1.13 (PD7(AIN1)), P1.8 (P8): now also P7.1 (P1)
- net at C4.2, D3.2: now also K1.1
- net at C4.1, D3.4: now also K1.2, K1.3
- new net: D5.2 (K), P6.3 (P3), R4.2, R6.2
- new net: D4.2 (K), P6.2 (P2), R3.1, R5.2
- new net USBVCC: C10.1, P6.1 (P1), R3.2
Other:
- moved on the sheet: C1, C2, C3, C4, C7, D2, IC1, P1, P2, P4, P5, R1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
