File: duin/duin.sch (KiCad schematic (older format))
At the start: 33 parts, among them IC1 ATMEGA8-PU, K1 JACK_2P, P1 ADC, P2 CONN_8, P3 CONN_6, P4 CONN_6, P5 CONN_3X2, P6 USB, P7 CONN_2, SW1 DPST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

Commit message: duin
Parts:
- removed C8, C9: C, symbol C
- removed U2: LD2903, symbol LM7805
- added C11: C, symbol C
- C1, C2: value C -> 22p
- C10: value CP -> 10uF
- C3: value C -> 100n
- D4, D5: value ZENER -> 3v6
- P7: value CONN_2 -> BOOTLOADER; symbol CONN_2 -> CONN_3
- R1: value R -> 10k
- R2: value R -> 1k
- X1: value CRYSTAL -> 16MHz
Connections:
- net +3.3V: no longer C7.1, IC1.20 (AVCC)
- net +5V: now also C7.1, IC1.20 (AVCC), P5.2, C11.1
- net GND: now also P5.6, P7.3 (P3), C11.2; no longer P7.2 (PM)
- net PD4: now also R5.2; no longer R5.1
- net RESET: now also P5.5
- net at IC1.13 (PD7(AIN1)), P1.8 (P8), P7.1 (P1): now also P7.2 (PM)
- net MOSI: now reaches IC1.17 (PB3(MOSI/OC2)), P2.4 (P4)
- net MOSI: now also P5.4
- net MISO: now reaches IC1.18 (PB4(MISO)), P2.5 (P5)
- net MISO: now also P5.1
- net SCK: now reaches IC1.19 (PB5(SCK)), P2.6 (P6), R2.1
- net SCK: now also P5.3
- net at D4.2 (K), P6.2 (P2), R3.1: now also R5.1; no longer R5.2
Other:
- moved on the sheet: C1, C2, C3, C7, D2, IC1, P1, P2, P4, P5, R1, R2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

Commit message: usbnoobie, ty! and some stickers
Parts:
- X1: value 16MHz -> 16..20MHz
Connections:
- net PD7: now reaches IC1.13 (PD7(AIN1)), P1.8 (P8), P7.1 (P1), P7.2 (PM)
- net PD7: now also R5.2
- net PD4: no longer names the net of IC1.6 (PD4(T0/XCK)), P1.5 (P5)
- net PD4: no longer R5.2
Changed lines of the file:
@@
-EESchema Schematic File Version 2  date Thu 23 Dec 2010 07:54:54 AM BRST
+EESchema Schematic File Version 2  date Fri 24 Dec 2010 10:08:35 PM BRST
 LIBS:power
 LIBS:device
@@
 Sheet 1 1
 Title ""
-Date "23 dec 2010"
+Date "25 dec 2010"
 Rev ""
 Comp ""
@@
 Comment4 ""
 $EndDescr
+Wire Wire Line
+	7750 4650 6950 4650
 Connection ~ 8300 5600
 Wire Wire Line
@@
 Connection ~ 7500 3950
 Wire Wire Line
-	7500 3850 7500 4750
+	7500 4750 7500 3850
 Connection ~ 6000 1150
 Connection ~ 1300 1350
@@
 Connection ~ 1900 6550
 Connection ~ 7500 4750
-Connection ~ 7750 4450
-Wire Wire Line
-	8300 4450 6950 4450
 Wire Wire Line
 	3200 5950 3600 5950
@@
 Connection ~ 2150 6050
 Wire Wire Line
-	2700 6050 1650 6050
+	1650 6050 2700 6050
 Wire Wire Line
 	1900 5950 1900 6150
 Wire Wire Line
-	1650 6150 1650 6650
+	1650 6650 1650 6150
 Connection ~ 1650 6550
 Connection ~ 6550 1550
@@
 Wire Wire Line
 	7750 4050 6950 4050
-Wire Wire Line
-	6950 4650 7750 4650
 Wire Wire Line
 	6950 4950 7650 4950
@@
 Connection ~ 5550 1550
 Wire Wire Line
-	5400 1150 6800 1150
+	6800 1150 5400 1150
 Connection ~ 4200 1550
 Wire Wire Line
 	4150 2500 4150 2650
 Wire Wire Line
-	4550 3150 4150 3150
+	4150 3150 4550 3150
 Wire Wire Line
 	3800 4650 4550 4650
@@
 	4200 3550 3900 3550
 Wire Wire Line
-	3500 3550 3500 4150
-Wire Wire Line
-	4550 5350 4550 5150
+	3500 4150 3500 3550
+Wire Wire Line
+	4550 5150 4550 5350
 Wire Wire Line
 	4550 4250 4250 4250
@@
 Connection ~ 5000 1550
 Wire Wire Line
-	5500 2650 5500 2250
+	5500 2250 5500 2650
 Wire Wire Line
 	7350 5700 7750 5700
@@
 Wire Wire Line
 	7600 5050 6950 5050
-Wire Wire Line
-	7750 4750 6950 4750
 Wire Wire Line
 	7750 4550 6950 4550
@@
 	2150 6150 2150 6050
 Wire Wire Line
-	2700 5950 1650 5950
+	1650 5950 2700 5950
 Connection ~ 1900 5950
 Wire Wire Line
-	1650 6550 2400 6550
+	2400 6550 1650 6550
 Connection ~ 2150 6550
 Wire Wire Line
@@
 	3400 6050 3200 6050
 Wire Wire Line
-	8300 4250 6950 4250
+	6950 4250 8300 4250
 Connection ~ 7750 4250
 Wire Wire Line
@@
 	8350 4950 8350 5500
 Connection ~ 8350 5500
+Wire Wire Line
+	7750 4450 6950 4450
+Wire Wire Line
+	8300 4750 6950 4750
+Connection ~ 7750 4750
 Text GLabel 9900 2400 2    60   Input ~ 0
 +5V
@@
 	-1   0    0    1
 $EndComp
-Text GLabel 8300 4450 2    60   Input ~ 0
-PD4
+Text GLabel 8300 4750 2    60   Input ~ 0
+PD7
 Text GLabel 8300 4250 2    60   Input ~ 0
 PD2
@@
 PD2
 Text GLabel 3600 5950 3    60   Input ~ 0
-PD4
+PD7
 $Comp
 L GND #PWR03
@@
 P 3900 3850
 F 0 "X1" H 3900 4000 60  0000 C CNN
-F 1 "16MHz" H 3900 3700 60  0000 C CNN
+F 1 "16..20MHz" H 3900 3700 60  0000 C CNN
 	1    3900 3850
 	0    1    1    0

Commit message: duin aref fix
Parts:
- C7: value C -> 100n
Connections:
- net +5V: no longer C7.1
- net GND: now also C7.1
Changed lines of the file:
@@
-EESchema Schematic File Version 2  date Fri 24 Dec 2010 10:08:35 PM BRST
+EESchema Schematic File Version 2  date Tue 04 Jan 2011 02:59:15 AM BRST
 LIBS:power
 LIBS:device
@@
 Sheet 1 1
 Title ""
-Date "25 dec 2010"
+Date "4 jan 2011"
 Rev ""
 Comp ""
@@
 Comment4 ""
 $EndDescr
+Text GLabel 6950 6450 0    60   Input ~ 0
+GND
 Wire Wire Line
 	7750 4650 6950 4650
@@
 Text GLabel 5800 1150 1    60   Input ~ 0
 +5V
-Text GLabel 6950 6450 2    60   Input ~ 0
-+5V
 $Comp
 L C C7
@@
 P 6950 6100
 F 0 "C7" H 7000 6200 50  0000 L CNN
-F 1 "C" H 7000 6000 50  0000 L CNN
+F 1 "100n" H 7000 6000 50  0000 L CNN
 	1    6950 6100
 	-1   0    0    1
